File: kicad_docs/_autosave-haible_2040_LPF_plug_in_board.kicad_pcb (KiCad board)
At the start: 2 copper layers, 58.4 x 50.8 mm, 96 parts, among them J1 Conn_01x04_Male, J2 Conn_01x04_Male, J3 Conn_01x04_Male, J4 Conn_01x08_Male, Q1 BCM857DS, Q10 BCM847DS, Q11 BC847, Q12 BCM847DS, Q13 BCM857DS, Q14 BCM847DS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

Commit message: tidy up pcb
Routing:
- net Net-(C4-Pad2): track 54.9 -> 45.9 mm
- net GND: vias 76 -> 74
Other:
- board text added: "+12V"
- board text added: "-12V"
- board text added: "cv in"
- board text added: "github.com/JordanAceto/haible_2040_LPF_plug_in_board rev 1 2020/02/02"
- board text added: "gnd"
- board text added: "rez cv in"
- board text added: "signal in"
- board text added: "signal out"
